Commit message: Edited xacro file

File: robot_description/urdf/thaara_mol.xacro (robot description, xacro)
@@ -136,5 +136,5 @@
     <inertial><origin xyz="0 0 0"/><mass value="0.2"/><inertia ixx="0.001" ixy="0.0" ixz="0.0" iyy="0.001" iyz="0.0" izz="0.001"/></inertial>
     <visual><origin xyz="0.0 -0.1905 0.03175"/><geometry><mesh filename="package://robot_description/meshes/head_v4.stl" scale="${mesh_scale} ${mesh_scale} ${mesh_scale}"/></geometry></visual>
-    <collision><origin xyz="0 0 0"/><geometry><box size="0 0 0"/></geometry></collision>
+    <collision><origin xyz="0 0 0"/><geometry><box size="0.05 0.05 0.05"/></geometry></collision>
   </link>
   <xacro:hand_link name="hand_1" xyz="0 0 -0.34925" rpy="${pos} 0 ${pos}"/>
